Commit message: modified:   src/isaacsim/scripts/standalone/task.py 	modified:   src/tamp/content/assets/robot/dcp_description/urdf/gripper/2f_85.urdf 	renamed:    src/tamp/content/assets/robot/dcp_description/urdf/gripper/vgc10_1cup.urdf -> src/tamp/content/assets/robot/dcp_description/urdf/gripper/vgc10.urdf 	deleted:    src/tamp/content/assets/robot/dcp_description/urdf/gripper/vgc10_4cups.urdf 	new file:   src/tamp/content/assets/robot/dcp_description/usd/gripper_visual/2f_85.usd 	new file:   src/tamp/content/assets/robot/dcp_description/usd/gripper_visual/2f_85/2f_85.usd 	new file:   src/tamp/content/assets/robot/dcp_description/usd/gripper_visual/2f_85/configuration/2f_85_base.usd 	new file:   src/tamp/content/assets/robot/dcp_description/usd/gripper_visual/2f_85/configuration/2f_85_physics.usd 	new file:   src/tamp/content/assets/robot/dcp_description/usd/gripper_visual/2f_85/configuration/2f_85_robot.usd 	new file:   src/tamp/content/assets/robot/dcp_description/usd/gripper_visual/2f_85/configuration/2f_85_sensor.usd 	new file:   src/tamp/content/assets/robot/dcp_description/usd/gripper_visual/ag95/ag95.usd 	new file:   src/tamp/content/assets/robot/dcp_description/usd/gripper_visual/ag95/configuration/ag95_base.usd 	new file:   src/tamp/content/assets/robot/dcp_description/usd/gripper_visual/ag95/configuration/ag95_physics.usd 	new file:   src/tamp/content/assets/robot/dcp_description/usd/gripper_visual/ag95/configuration/ag95_robot.usd 	new file:   src/tamp/content/assets/robot/dcp_description/usd/gripper_visual/ag95/configuration/ag95_sensor.usd 	new file:   src/tamp/content/assets/robot/dcp_description/usd/gripper_visual/vgc10/configuration/vgc10_base.usd 	new file:   src/tamp/content/assets/robot/dcp_description/usd/gripper_visual/vgc10/configuration/vgc10_physics.usd 	new file:   src/tamp/content/assets/robot/dcp_description/usd/gripper_visual/vgc10/configuration/vgc10_robot.usd 	new file:   src/tamp/content/assets/robot/dcp_description/usd/gripper_visual/vgc10/configuration/vgc10_sensor.usd 	new file:   src/tamp/content/assets/robot/dcp_description/usd/gripper_visual/vgc10/vgc10.usd

File: src/tamp/content/assets/robot/dcp_description/urdf/gripper/2f_85.urdf (robot description, URDF)
Before this commit: robot robotiq_gripper, 9 links, 8 joints
Links:
- link robotiq_85_base_link: geometry collision mesh filename=package://dcp_description/meshes/gripper/2f_85/collision/ro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; visual mesh filename=package://dcp_description/meshes/gripper/2f_85/visual/robot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
- link robotiq_85_left_finger_link: geometry collision mesh filename=package://dcp_description/meshes/gripper/2f_85/collision/le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; visual mesh filename=package://dcp_description/meshes/gripper/2f_85/visual/left_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
- link robotiq_85_left_finger_tip_link: geometry collision mesh filename=package://dcp_description/meshes/gripper/2f_85/collision/le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; visual mesh filename=package://dcp_description/meshes/gripper/2f_85/visual/left_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
- link robotiq_85_left_inner_knuckle_link: geometry collision mesh filename=package://dcp_description/meshes/gripper/2f_85/collision/le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; visual mesh filename=package://dcp_description/meshes/gripper/2f_85/visual/left_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
- link robotiq_85_left_knuckle_link: geometry collision mesh filename=package://dcp_description/meshes/gripper/2f_85/collision/le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; visual mesh filename=package://dcp_description/meshes/gripper/2f_85/visual/left_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
- link robotiq_85_right_finger_link: geometry collision mesh filename=package://dcp_description/meshes/gripper/2f_85/collision/ri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; visual mesh filename=package://dcp_description/meshes/gripper/2f_85/visual/right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
- link robotiq_85_right_finger_tip_link: geometry collision mesh filename=package://dcp_description/meshes/gripper/2f_85/collision/ri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; visual mesh filename=package://dcp_description/meshes/gripper/2f_85/visual/right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
- link robotiq_85_right_inner_knuckle_link: geometry collision mesh filename=package://dcp_description/meshes/gripper/2f_85/collision/ri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; visual mesh filename=package://dcp_description/meshes/gripper/2f_85/visual/right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
- link robotiq_85_right_knuckle_link: geometry collision mesh filename=package://dcp_description/meshes/gripper/2f_85/collision/ri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; visual mesh filename=package://dcp_description/meshes/gripper/2f_85/visual/right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
