Commit message: 수정함:        src/cuTAMP/cutamp/robots/assets/fr5_vgc10.yml 	수정함:        src/isaacsim/scripts/standalone/task.py 	수정함:        src/tamp/content/assets/robot/dcp_description/urdf/gripper/vgc10.urdf 	수정함:        src/tamp/content/assets/robot/dcp_description/urdf/robot/fr5_vgc10.urdf 	수정함:        src/tamp/content/assets/robot/dcp_description/usd/fr5_vgc10/configuration/fr5_vgc10_base.usd 	수정함:        src/tamp/content/assets/robot/dcp_description/usd/fr5_vgc10/configuration/fr5_vgc10_physics.usd 	수정함:        src/tamp/content/assets/robot/dcp_description/usd/fr5_vgc10/configuration/fr5_vgc10_robot.usd 	수정함:        src/tamp/content/assets/robot/dcp_description/usd/fr5_vgc10/fr5_vgc10.usd 	수정함:        src/tamp/content/assets/robot/dcp_description/usd/gripper_visual/vgc10/configuration/vgc10_base.usd 	수정함:        src/tamp/content/assets/robot/dcp_description/usd/gripper_visual/vgc10/configuration/vgc10_physics.usd 	수정함:        src/tamp/content/assets/robot/dcp_description/usd/gripper_visual/vgc10/configuration/vgc10_robot.usd 	수정함:        src/tamp/content/assets/robot/dcp_description/usd/gripper_visual/vgc10/vgc10.usd 	수정함:        src/tamp/content/configs/robot/spheres/fr5_vgc10.yml 	수정함:        src/tamp/scripts/client/tamp_client.py

File: src/tamp/content/assets/robot/dcp_description/urdf/gripper/vgc10.urdf (robot description, URDF)
Before this commit: robot onrobot_vgc10_model, 2 links, 1 joints
Links:
- removed link onrobot_vgc10_base_link
- added link gripper_base_link, mass 0.6; collision mesh filename=package://dcp_description/meshes/gripper/vgc10/collision/ba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; visual mesh filename=package://dcp_description/meshes/gripper/vgc10/visual/base_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
Joints:
- joint suction_joint: parent onrobot_vgc10_base_link -> gripper_base_link

File: src/tamp/content/assets/robot/dcp_description/urdf/robot/fr5_vgc10.urdf (robot description, URDF)
Before this commit: robot fr5_ag95, 11 links, 10 joints
Links:
- removed link onrobot_vgc10_base_link
- added link grasp_frame, mass 0.01
- added link gripper_base_link, mass 0.6; collision mesh filename=package://dcp_description/meshes/gripper/vgc10/collision/ba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; visual mesh filename=package://dcp_description/meshes/gripper/vgc10/visual/base_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
Joints:
- removed joint onrobot_vgc10_base_joint
- added joint grasp_joint: type fixed, parent gripper_base_link, child grasp_frame, origin xyz=0 0 0.18 rpy=0 0 0.0, axis 0 0 1
- added joint gripper_base_joint: type fixed, parent tool0, child gripper_base_link, origin xyz=0 0 0 rpy=0 0 0
- joint suction_joint: parent onrobot_vgc10_base_link -> gripper_base_link
