Commit message: 수정함:        src/tamp/content/assets/robot/dcp_description/urdf/robot/fr5_2f_85.urdf 	수정함:        src/tamp/content/assets/robot/dcp_description/usd/fr5_2f_85/fr5_2f_85.usd 	수정함:        src/tamp/scripts/client/tamp_client.py 	수정함:        src/tamp/scripts/server/tamp_server.py 	수정함:        src/tamp_interfaces/CMakeLists.txt 	새 파일:       src/tamp_interfaces/srv/SetTampCfg.srv

File: src/tamp/content/assets/robot/dcp_description/urdf/robot/fr5_2f_85.urdf (robot description, URDF)
Before this commit: robot fr5_ag95, 20 links, 19 joints
Joints:
- joint grasp_joint: origin xyz=0 0 0.15 rpy=0 0 0 -> xyz=0 0 0.1 rpy=0 0 0
